Commit message: try editing urdf

File: src/urg_node/urdf/hokuyo_ust10.urdf.xacro (robot description, xacro)
@@ -51,22 +51,8 @@
     </xacro:macro>
     <xacro:hokuyo_ust10 frame="laser" topic="${topic}"/>
-    <joint name="laser_mount_joint" type="fixed">
-      <xacro:insert_block name="origin" />
-      <parent link="${parent_link}" />
-      <child link="laser_mount" />
-    </joint>
-    <link name="laser_mount">
-      <visual>
-        <origin xyz="0 0 0" rpy="0 0 0" />
-        <geometry>
-          <!-- Origin of this mesh is the base of the bracket. -->
-          <mesh filename="package://urg_node/meshes/hokuyo_ust10.stl" />
-        </geometry>
-      </visual>
-    </link>
     <joint name="laser_joint" type="fixed">
       <!-- This offset is from the base of the bracket to the LIDAR's focal point. -->
       <origin xyz="0 0 0.0474" rpy="0 0 0" />
-      <parent link="laser_mount" />
+      <parent link="base_link" />
       <child link="laser" />
     </joint>

Commit message: try adding base_footprint

File: src/urg_node/urdf/hokuyo_ust10.urdf.xacro (robot description, xacro)
@@ -70,4 +70,12 @@
     </visual>
   </link>
+    <!-- BASE_FOOTPRINT LINK -->
+    <joint name="base_footprint_joint" type="fixed">
+        <parent link="base_link"/>
+        <child link="base_footprint"/>
+        <origin xyz="0 0 0" rpy="0 0 0"/>
+    </joint>
+    <link name="base_footprint">
+    </link>
     <xacro:hokuyo_ust10_mount prefix="" topic="scan" parent_link="base_link" min_angle="-2.35619" max_angle="2.35619">
   <origin xyz="0 0 0.1" rpy="0 0 0" />
